File: PCB/EtchPad.kicad_pcb (KiCad board)
At the start: 2 copper layers, 81 x 50.6 mm, 12 parts, among them SW1 SW_Push, SW2 SW_Push, SW3 SW_Push, SW4 SW_Push, SW5 RotaryEncoder_Switch, SW6 RotaryEncoder_Switch, U1 XIAO-RP2040-DIP

Commit message: Add files via upload
Parts:
- moved D1 4.76 mm to (52.4, 121.4)
- moved D2 4.76 mm to (71.4, 121.4)
- moved D3 4.76 mm to (90.5, 121.4)
- moved D4 4.76 mm to (109.5, 121.4)
Routing:
- net GND: track 307.6 -> 258.9 mm, vias 7 -> 4
- net Net-(D1-DOUT): track 37.7 -> 51.2 mm, vias 0 -> 2
- net +5V: track 121.3 -> 110.5 mm, vias 3 -> 1
- net Net-(D2-DOUT): track 44.5 -> 37.0 mm
- net Net-(D3-DOUT): track 42.8 -> 38.3 mm
- net Net-(D1-DIN): track 38.0 -> 41.5 mm
Other:
- board text added: "The Opposite Of: Always, Coming, From, Take, Me, Down"
